File: hardware/motor-control-board/circuit/power-delivery/CYPD-3177 Breakout.kicad_sch (KiCad schematic)
At the start: 25 parts, among them J1 USB-C Power, J2 Conn_01x12, J4 Conn_01x12, Q1 DMP3013SFV, Q2 DMP3013SFV, U1 CYPD3177

Commit message: re-laid out and re-routed PCB - V1.0 ready for production
Parts:
- J1: footprint Connector_USB:USB_C_Receptacle_HRO_TYPE-C-31-M-12 -> Library:USB-C-SMD_MC-311D

Commit message: edited USB-C connector footprint to match chosen component - plus other misc DRC fixes - ready for production - some manual adjustment still needed (U1 orientation, USB-C position wrong etc
Parts:
- J1: footprint Library:USB-C-SMD_MC-311D -> Library:SOFNG_MC-311D_12P_Female_USB-C_Connector
Changed lines of the file:
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@@
 			)
 		)
-		(property "Footprint" "Library:USB-C-SMD_MC-311D"
+		(property "Footprint" "Library:SOFNG_MC-311D_12P_Female_USB-C_Connector"
 			(at 35.56 43.18 0)
 			(effects
